Commit message: moved sciurus robot meshes into subdirectory

File: sciurus17_description/urdf/sciurus17/sciurus17_body.xacro (robot description, xacro)
@@ -13,5 +13,5 @@
       <visual>
         <geometry>
-          <mesh filename="package://sciurus17_description/meshes/visual/Base.stl" scale="1.0 1.0 1.0"/>
+          <mesh filename="package://sciurus17_description/meshes/sciurus17/visual/Base.stl" scale="1.0 1.0 1.0"/>
         </geometry>
         <material name="${base_color}"/>
@@ -20,5 +20,5 @@
         <origin rpy="0 0 0" xyz="0.0 0.0 0.0"/>
         <geometry>
-          <mesh filename="package://sciurus17_description/meshes/collision/Base.stl" scale="1.0 1.0 1.0"/>
+          <mesh filename="package://sciurus17_description/meshes/sciurus17/collision/Base.stl" scale="1.0 1.0 1.0"/>
         </geometry>
       </collision>
@@ -44,5 +44,5 @@
       <visual>
         <geometry>
-          <mesh filename="package://sciurus17_description/meshes/visual/Body.stl" scale="1.0 1.0 1.0"/>
+          <mesh filename="package://sciurus17_description/meshes/sciurus17/visual/Body.stl" scale="1.0 1.0 1.0"/>
         </geometry>
         <material name="${body_color}"/>
@@ -51,5 +51,5 @@
         <origin rpy="0 0 0" xyz="0.0 0.0 0.0"/>
         <geometry>
-          <mesh filename="package://sciurus17_description/meshes/collision/Body.stl" scale="1.0 1.0 1.0"/>
+          <mesh filename="package://sciurus17_description/meshes/sciurus17/collision/Body.stl" scale="1.0 1.0 1.0"/>
         </geometry>
       </collision>

File: sciurus17_description/urdf/sciurus17/sciurus17_head.xacro (robot description, xacro)
@@ -26,5 +26,5 @@
       <visual>
         <geometry>
-          <mesh filename="package://sciurus17_description/meshes/visual/Neck1.stl" scale="1.0 1.0 1.0"/>
+          <mesh filename="package://sciurus17_description/meshes/sciurus17/visual/Neck1.stl" scale="1.0 1.0 1.0"/>
         </geometry>
         <material name="${head_color}"/>
@@ -32,5 +32,5 @@
       <collision>
         <geometry>
-          <mesh filename="package://sciurus17_description/meshes/collision/Neck1.stl" scale="1.0 1.0 1.0"/>
+          <mesh filename="package://sciurus17_description/meshes/sciurus17/collision/Neck1.stl" scale="1.0 1.0 1.0"/>
         </geometry>
       </collision>
@@ -57,5 +57,5 @@
         <origin rpy="1.5708 0 0" xyz="0.0 0.0 0.0"/>
         <geometry>
-          <mesh filename="package://sciurus17_description/meshes/visual/Neck2.stl" scale="1.0 1.0 1.0"/>
+          <mesh filename="package://sciurus17_description/meshes/sciurus17/visual/Neck2.stl" scale="1.0 1.0 1.0"/>
         </geometry>
         <material name="${head_color}"/>
@@ -64,5 +64,5 @@
         <origin rpy="1.5708 0 0" xyz="0.0 0.0 0.0"/>
         <geometry>
-          <mesh filename="package://sciurus17_description/meshes/collision/Neck2.stl" scale="1.0 1.0 1.0"/>
+          <mesh filename="package://sciurus17_description/meshes/sciurus17/collision/Neck2.stl" scale="1.0 1.0 1.0"/>
         </geometry>
       </collision>

File: sciurus17_description/urdf/sciurus17/sciurus17_left_arm.xacro (robot description, xacro)
@@ -36,12 +36,12 @@
         <origin rpy="-1.5708 0 0" xyz="0.0 0.0 0.0"/>
         <geometry>
-          <mesh filename="package://sciurus17_description/meshes/visual/L_Link1.stl" scale="1.0 1.0 1.0"/>
-        </geometry>
-        <material name="${arm_color}"/>
-      </visual>
-      <collision>
-        <origin rpy="-1.5708 0 0" xyz="0.0 0.0 0.0"/>
-        <geometry>
-          <mesh filename="package://sciurus17_description/meshes/collision/L_Link1.stl" scale="1.0 1.0 1.0"/>
+          <mesh filename="package://sciurus17_description/meshes/sciurus17/visual/L_Link1.stl" scale="1.0 1.0 1.0"/>
+        </geometry>
+        <material name="${arm_color}"/>
+      </visual>
+      <collision>
+        <origin rpy="-1.5708 0 0" xyz="0.0 0.0 0.0"/>
+        <geometry>
+          <mesh filename="package://sciurus17_description/meshes/sciurus17/collision/L_Link1.stl" scale="1.0 1.0 1.0"/>
         </geometry>
       </collision>
@@ -68,5 +68,5 @@
         <origin rpy="0 -1.5708 0" xyz="0.0 0.0 0.0"/>
         <geometry>
-          <mesh filename="package://sciurus17_description/meshes/visual/L_Link2.stl" scale="-1.0 1.0 -1.0"/>
+          <mesh filename="package://sciurus17_description/meshes/sciurus17/visual/L_Link2.stl" scale="-1.0 1.0 -1.0"/>
         </geometry>
         <material name="${arm_color}"/>
@@ -75,5 +75,5 @@
         <origin rpy="0 -1.5708 0" xyz="0.0 0.0 0.0"/>
         <geometry>
-          <mesh filename="package://sciurus17_description/meshes/collision/L_Link2.stl" scale="-1.0 1.0 -1.0"/>
+          <mesh filename="package://sciurus17_description/meshes/sciurus17/collision/L_Link2.stl" scale="-1.0 1.0 -1.0"/>
         </geometry>
       </collision>
@@ -100,12 +100,12 @@
         <origin rpy="-1.5708 0 0" xyz="0.0 0.0 0.0"/>
         <geometry>
-          <mesh filename="package://sciurus17_description/meshes/visual/L_Link3.stl" scale="1.0 1.0 1.0"/>
-        </geometry>
-        <material name="${arm_color}"/>
-      </visual>
-      <collision>
-        <origin rpy="-1.5708 0 0" xyz="0.0 0.0 0.0"/>
-        <geometry>
-          <mesh filename="package://sciurus17_description/meshes/collision/L_Link3.stl" scale="1.0 1.0 1.0"/>
+          <mesh filename="package://sciurus17_description/meshes/sciurus17/visual/L_Link3.stl" scale="1.0 1.0 1.0"/>
+        </geometry>
+        <material name="${arm_color}"/>
+      </visual>
+      <collision>
+        <origin rpy="-1.5708 0 0" xyz="0.0 0.0 0.0"/>
+        <geometry>
+          <mesh filename="package://sciurus17_description/meshes/sciurus17/collision/L_Link3.stl" scale="1.0 1.0 1.0"/>
         </geometry>
       </collision>
@@ -132,12 +132,12 @@
         <origin rpy="0 0 0" xyz="0.0 0.0 0.0"/>
         <geometry>
-          <mesh filename="package://sciurus17_description/meshes/visual/L_Link4.stl" scale="1.0 1.0 1.0"/>
-        </geometry>
-        <material name="${arm_color}"/>
-      </visual>
-      <collision>
-        <origin rpy="0 0 0" xyz="0.0 0.0 0.0"/>
-        <geometry>
-          <mesh filename="package://sciurus17_description/meshes/collision/L_Link4.stl" scale="1.0 1.0 1.0"/>
+          <mesh filename="package://sciurus17_description/meshes/sciurus17/visual/L_Link4.stl" scale="1.0 1.0 1.0"/>
+        </geometry>
+        <material name="${arm_color}"/>
+      </visual>
+      <collision>
+        <origin rpy="0 0 0" xyz="0.0 0.0 0.0"/>
+        <geometry>
+          <mesh filename="package://sciurus17_description/meshes/sciurus17/collision/L_Link4.stl" scale="1.0 1.0 1.0"/>
         </geometry>
       </collision>
@@ -164,5 +164,5 @@
         <origin rpy="-1.5708 0 0" xyz="0.0 0.0 0.0"/>
         <geometry>
-          <mesh filename="package://sciurus17_description/meshes/visual/L_Link5.stl" scale="1.0 1.0 1.0"/>
+          <mesh filename="package://sciurus17_description/meshes/sciurus17/visual/L_Link5.stl" scale="1.0 1.0 1.0"/>
         </geometry>
         <material name="${arm_color}"/>
@@ -171,5 +171,5 @@
         <origin xyz="0.032 0.074 -0.0346" rpy="3.1415926 0 2.0944"/>
         <geometry>
-          <mesh filename="package://sciurus17_description/meshes/visual/Logo_Rabbit.stl" scale="1.0 1.0 1.0"/>
+          <mesh filename="package://sciurus17_description/meshes/sciurus17/visual/Logo_Rabbit.stl" scale="1.0 1.0 1.0"/>
         </geometry>
         <material name="red_color">
@@ -180,5 +180,5 @@
         <origin xyz="0.013 0.107 -0.0346" rpy="3.1415926 0 2.0944"/>
         <geometry>
-          <mesh filename="package://sciurus17_description/meshes/visual/Logo_Corp.stl" scale="1.0 1.0 1.0"/>
+          <mesh filename="package://sciurus17_description/meshes/sciurus17/visual/Logo_Corp.stl" scale="1.0 1.0 1.0"/>
         </geometry>
         <material name="black_color">
@@ -189,5 +189,5 @@
         <origin rpy="-1.5708 0 0" xyz="0.0 0.0 0.0"/>
         <geometry>
-          <mesh filename="package://sciurus17_description/meshes/collision/L_Link5.stl" scale="1.0 1.0 1.0"/>
+          <mesh filename="package://sciurus17_description/meshes/sciurus17/collision/L_Link5.stl" scale="1.0 1.0 1.0"/>
         </geometry>
       </collision>
@@ -211,4 +211,10 @@
         <material name="${arm_color}"/>
       </visual>
+      <collision>
+        <origin rpy="0 0 0" xyz="0.0 0.0 0.0"/>
+        <geometry>
+          <cylinder length="0.001" radius="0.001"/>
+        </geometry>
+      </collision>
     </link>
     <joint name="l_arm_joint6" type="revolute">
@@ -228,12 +234,12 @@
         <origin rpy="0 0 0" xyz="0.0 0.0 0.0"/>
         <geometry>
-          <mesh filename="package://sciurus17_description/meshes/visual/L_Link6.stl" scale="1.0 1.0 1.0"/>
-        </geometry>
-        <material name="${arm_color}"/>
-      </visual>
-      <collision>
-        <origin rpy="0 0 0" xyz="0.0 0.0 0.0"/>
-        <geometry>
-          <mesh filename="package://sciurus17_description/meshes/collision/L_Link6.stl" scale="1.0 1.0 1.0"/>
+          <mesh filename="package://sciurus17_description/meshes/sciurus17/visual/L_Link6.stl" scale="1.0 1.0 1.0"/>
+        </geometry>
+        <material name="${arm_color}"/>
+      </visual>
+      <collision>
+        <origin rpy="0 0 0" xyz="0.0 0.0 0.0"/>
+        <geometry>
+          <mesh filename="package://sciurus17_description/meshes/sciurus17/collision/L_Link6.stl" scale="1.0 1.0 1.0"/>
         </geometry>
       </collision>

File: sciurus17_description/urdf/sciurus17/sciurus17_left_hand.xacro (robot description, xacro)
@@ -12,5 +12,5 @@
         <origin rpy="1.5708 0 0" xyz="0.0 0.0 0.0"/>
         <geometry>
-          <mesh filename="package://sciurus17_description/meshes/visual/L_Link7.stl" scale="1.0 1.0 1.0"/>
+          <mesh filename="package://sciurus17_description/meshes/sciurus17/visual/L_Link7.stl" scale="1.0 1.0 1.0"/>
         </geometry>
         <material name="${hand_color}"/>
@@ -19,5 +19,5 @@
         <origin rpy="1.5708 0 0" xyz="0.0 0.0 0.0"/>
         <geometry>
-          <mesh filename="package://sciurus17_description/meshes/collision/L_Link7.stl" scale="1.0 1.0 1.0"/>
+          <mesh filename="package://sciurus17_description/meshes/sciurus17/collision/L_Link7.stl" scale="1.0 1.0 1.0"/>
         </geometry>
       </collision>
@@ -44,5 +44,5 @@
         <origin rpy="0 0 0" xyz="0.0 0.0 0.0"/>
         <geometry>
-          <mesh filename="package://sciurus17_description/meshes/visual/L_HandA.stl" scale="1.0 1.0 1.0"/>
+          <mesh filename="package://sciurus17_description/meshes/sciurus17/visual/L_HandA.stl" scale="1.0 1.0 1.0"/>
         </geometry>
         <material name="${hand_color}"/>
@@ -51,5 +51,5 @@
         <origin rpy="0 0 0" xyz="0.0 0.0 0.0"/>
         <geometry>
-          <mesh filename="package://sciurus17_description/meshes/collision/L_HandA.stl" scale="1.0 1.0 1.0"/>
+          <mesh filename="package://sciurus17_description/meshes/sciurus17/collision/L_HandA.stl" scale="1.0 1.0 1.0"/>
         </geometry>
       </collision>
@@ -77,5 +77,5 @@
         <origin rpy="0 0 0" xyz="0.0 0.0 0.0"/>
         <geometry>
-          <mesh filename="package://sciurus17_description/meshes/visual/L_HandB.stl" scale="1.0 1.0 1.0"/>
+          <mesh filename="package://sciurus17_description/meshes/sciurus17/visual/L_HandB.stl" scale="1.0 1.0 1.0"/>
         </geometry>
         <material name="${hand_color}"/>
@@ -84,5 +84,5 @@
         <origin rpy="0 0 0" xyz="0.0 0.0 0.0"/>
         <geometry>
-          <mesh filename="package://sciurus17_description/meshes/collision/L_HandB.stl" scale="1.0 1.0 1.0"/>
+          <mesh filename="package://sciurus17_description/meshes/sciurus17/collision/L_HandB.stl" scale="1.0 1.0 1.0"/>
         </geometry>
       </collision>

File: sciurus17_description/urdf/sciurus17/sciurus17_right_arm.xacro (robot description, xacro)
@@ -36,12 +36,12 @@
         <origin rpy="1.5708 0 0" xyz="0.0 0.0 0.0"/>
         <geometry>
-          <mesh filename="package://sciurus17_description/meshes/visual/R_Link1.stl" scale="1.0 1.0 1.0"/>
-        </geometry>
-        <material name="${arm_color}"/>
-      </visual>
-      <collision>
-        <origin rpy="1.5708 0 0" xyz="0.0 0.0 0.0"/>
-        <geometry>
-          <mesh filename="package://sciurus17_description/meshes/collision/R_Link1.stl" scale="1.0 1.0 1.0"/>
+          <mesh filename="package://sciurus17_description/meshes/sciurus17/visual/R_Link1.stl" scale="1.0 1.0 1.0"/>
+        </geometry>
+        <material name="${arm_color}"/>
+      </visual>
+      <collision>
+        <origin rpy="1.5708 0 0" xyz="0.0 0.0 0.0"/>
+        <geometry>
+          <mesh filename="package://sciurus17_description/meshes/sciurus17/collision/R_Link1.stl" scale="1.0 1.0 1.0"/>
         </geometry>
       </collision>
@@ -68,5 +68,5 @@
         <origin rpy="0 1.5708 0" xyz="0.0 0.0 0.0"/>
         <geometry>
-          <mesh filename="package://sciurus17_description/meshes/visual/R_Link2.stl" scale="1.0 1.0 1.0"/>
+          <mesh filename="package://sciurus17_description/meshes/sciurus17/visual/R_Link2.stl" scale="1.0 1.0 1.0"/>
         </geometry>
         <material name="${arm_color}"/>
@@ -75,5 +75,5 @@
         <origin rpy="0 1.5708 0" xyz="0.0 0.0 0.0"/>
         <geometry>
-          <mesh filename="package://sciurus17_description/meshes/collision/R_Link2.stl" scale="1.0 1.0 1.0"/>
+          <mesh filename="package://sciurus17_description/meshes/sciurus17/collision/R_Link2.stl" scale="1.0 1.0 1.0"/>
         </geometry>
       </collision>
@@ -100,12 +100,12 @@
         <origin rpy="1.5708 0 0" xyz="0.0 0.0 0.0"/>
         <geometry>
-          <mesh filename="package://sciurus17_description/meshes/visual/L_Link3.stl" scale="1.0 -1.0 1.0"/>
-        </geometry>
-        <material name="${arm_color}"/>
-      </visual>
-      <collision>
-        <origin rpy="1.5708 0 0" xyz="0.0 0.0 0.0"/>
-        <geometry>
-          <mesh filename="package://sciurus17_description/meshes/collision/L_Link3.stl" scale="1.0 -1.0 1.0"/>
+          <mesh filename="package://sciurus17_description/meshes/sciurus17/visual/L_Link3.stl" scale="1.0 -1.0 1.0"/>
+        </geometry>
+        <material name="${arm_color}"/>
+      </visual>
+      <collision>
+        <origin rpy="1.5708 0 0" xyz="0.0 0.0 0.0"/>
+        <geometry>
+          <mesh filename="package://sciurus17_description/meshes/sciurus17/collision/L_Link3.stl" scale="1.0 -1.0 1.0"/>
         </geometry>
       </collision>
@@ -132,12 +132,12 @@
         <origin rpy="0 0 0" xyz="0.0 0.0 0.0"/>
         <geometry>
-          <mesh filename="package://sciurus17_description/meshes/visual/R_Link4.stl" scale="1.0 1.0 1.0"/>
-        </geometry>
-        <material name="${arm_color}"/>
-      </visual>
-      <collision>
-        <origin rpy="0 0 0" xyz="0.0 0.0 0.0"/>
-        <geometry>
-          <mesh filename="package://sciurus17_description/meshes/collision/R_Link4.stl" scale="1.0 1.0 1.0"/>
+          <mesh filename="package://sciurus17_description/meshes/sciurus17/visual/R_Link4.stl" scale="1.0 1.0 1.0"/>
+        </geometry>
+        <material name="${arm_color}"/>
+      </visual>
+      <collision>
+        <origin rpy="0 0 0" xyz="0.0 0.0 0.0"/>
+        <geometry>
+          <mesh filename="package://sciurus17_description/meshes/sciurus17/collision/R_Link4.stl" scale="1.0 1.0 1.0"/>
         </geometry>
       </collision>
@@ -164,5 +164,5 @@
         <origin rpy="1.5708 0 0" xyz="0.0 0.0 0.0"/>
         <geometry>
-          <mesh filename="package://sciurus17_description/meshes/visual/R_Link5.stl" scale="1.0 1.0 1.0"/>
+          <mesh filename="package://sciurus17_description/meshes/sciurus17/visual/R_Link5.stl" scale="1.0 1.0 1.0"/>
         </geometry>
         <material name="${arm_color}"/>
@@ -171,5 +171,5 @@
         <origin xyz="0.032 -0.074 0.0345" rpy="0 0 -2.0944"/>
         <geometry>
-          <mesh filename="package://sciurus17_description/meshes/visual/Logo_Rabbit.stl" scale="1.0 1.0 1.0"/>
+          <mesh filename="package://sciurus17_description/meshes/sciurus17/visual/Logo_Rabbit.stl" scale="1.0 1.0 1.0"/>
         </geometry>
         <material name="red_color">
@@ -180,5 +180,5 @@
         <origin xyz="0.013 -0.107 0.0345" rpy="0 0 -2.0944"/>
         <geometry>
-          <mesh filename="package://sciurus17_description/meshes/visual/Logo_Corp.stl" scale="1.0 1.0 1.0"/>
+          <mesh filename="package://sciurus17_description/meshes/sciurus17/visual/Logo_Corp.stl" scale="1.0 1.0 1.0"/>
         </geometry>
         <material name="black_color">
@@ -189,5 +189,5 @@
         <origin rpy="1.5708 0 0" xyz="0.0 0.0 0.0"/>
         <geometry>
-          <mesh filename="package://sciurus17_description/meshes/collision/R_Link5.stl" scale="1.0 1.0 1.0"/>
+          <mesh filename="package://sciurus17_description/meshes/sciurus17/collision/R_Link5.stl" scale="1.0 1.0 1.0"/>
         </geometry>
       </collision>
@@ -211,4 +211,10 @@
         <material name="${arm_color}"/>
       </visual>
+      <collision>
+        <origin rpy="0 0 0" xyz="0.0 0.0 0.0"/>
+        <geometry>
+          <cylinder length="0.001" radius="0.001"/>
+        </geometry>
+      </collision>
     </link>
     <joint name="r_arm_joint6" type="revolute">
@@ -228,12 +234,12 @@
         <origin rpy="0 0 0" xyz="0.0 0.0 0.0"/>
         <geometry>
-          <mesh filename="package://sciurus17_description/meshes/visual/R_Link6.stl" scale="1.0 1.0 1.0"/>
-        </geometry>
-        <material name="${arm_color}"/>
-      </visual>
-      <collision>
-        <origin rpy="0 0 0" xyz="0.0 0.0 0.0"/>
-        <geometry>
-          <mesh filename="package://sciurus17_description/meshes/collision/R_Link6.stl" scale="1.0 1.0 1.0"/>
+          <mesh filename="package://sciurus17_description/meshes/sciurus17/visual/R_Link6.stl" scale="1.0 1.0 1.0"/>
+        </geometry>
+        <material name="${arm_color}"/>
+      </visual>
+      <collision>
+        <origin rpy="0 0 0" xyz="0.0 0.0 0.0"/>
+        <geometry>
+          <mesh filename="package://sciurus17_description/meshes/sciurus17/collision/R_Link6.stl" scale="1.0 1.0 1.0"/>
         </geometry>
       </collision>

File: sciurus17_description/urdf/sciurus17/sciurus17_right_hand.xacro (robot description, xacro)
@@ -12,5 +12,5 @@
         <origin rpy="1.5708 0 0" xyz="0.0 0.0 0.0"/>
         <geometry>
-          <mesh filename="package://sciurus17_description/meshes/visual/R_Link7.stl" scale="1.0 1.0 1.0"/>
+          <mesh filename="package://sciurus17_description/meshes/sciurus17/visual/R_Link7.stl" scale="1.0 1.0 1.0"/>
         </geometry>
         <material name="${hand_color}"/>
@@ -19,5 +19,5 @@
         <origin rpy="1.5708 0 0" xyz="0.0 0.0 0.0"/>
         <geometry>
-          <mesh filename="package://sciurus17_description/meshes/collision/R_Link7.stl" scale="1.0 1.0 1.0"/>
+          <mesh filename="package://sciurus17_description/meshes/sciurus17/collision/R_Link7.stl" scale="1.0 1.0 1.0"/>
         </geometry>
       </collision>
@@ -45,5 +45,5 @@
         <origin rpy="0 0 0" xyz="0.0 0.0 0.0"/>
         <geometry>
-          <mesh filename="package://sciurus17_description/meshes/visual/R_HandA.stl" scale="1.0 1.0 1.0"/>
+          <mesh filename="package://sciurus17_description/meshes/sciurus17/visual/R_HandA.stl" scale="1.0 1.0 1.0"/>
         </geometry>
         <material name="${hand_color}"/>
@@ -52,5 +52,5 @@
         <origin rpy="0 0 0" xyz="0.0 0.0 0.0"/>
         <geometry>
-          <mesh filename="package://sciurus17_description/meshes/collision/R_HandA.stl" scale="1.0 1.0 1.0"/>
+          <mesh filename="package://sciurus17_description/meshes/sciurus17/collision/R_HandA.stl" scale="1.0 1.0 1.0"/>
         </geometry>
       </collision>
@@ -79,5 +79,5 @@
         <origin rpy="0 0 0" xyz="0.0 0.0 0.0"/>
         <geometry>
-          <mesh filename="package://sciurus17_description/meshes/visual/R_HandB.stl" scale="1.0 1.0 1.0"/>
+          <mesh filename="package://sciurus17_description/meshes/sciurus17/visual/R_HandB.stl" scale="1.0 1.0 1.0"/>
         </geometry>
         <material name="${hand_color}"/>
@@ -86,5 +86,5 @@
         <origin rpy="0 0 0" xyz="0.0 0.0 0.0"/>
         <geometry>
-          <mesh filename="package://sciurus17_description/meshes/collision/R_HandB.stl" scale="1.0 1.0 1.0"/>
+          <mesh filename="package://sciurus17_description/meshes/sciurus17/collision/R_HandB.stl" scale="1.0 1.0 1.0"/>
         </geometry>
       </collision>

File: sciurus17_description/urdf/sciurus17/sciurus17_robot.urdf.xacro (robot description, xacro)
@@ -57,11 +57,11 @@
         <xacro:default_transmission joint_name="neck_pitch_joint"/>
       </xacro:if>
-      <!-- Used for fixing robot 'base_link'  to Gazebo 'world' -->
-      <link name="world"/>
-      <joint name="base_link_to_world_joint" type="fixed">
-        <parent link="world"/>
-        <child link="base_link"/>
-      </joint>
     </xacro:if>
+    <!-- Used for fixing robot 'base_link'  to Gazebo 'world' -->
+    <link name="world"/>
+    <joint name="base_link_to_world_joint" type="fixed">
+      <parent link="world"/>
+      <child link="base_link"/>
+    </joint>
     <xacro:sciurus17_body
       waist_yaw_upper_limit="${radians(-110)}"
@@ -76,5 +76,5 @@
       neck_yaw_upper_limit="${radians(165)}"
       neck_pitch_lower_limit="${radians(-90)}"
-      neck_pitch_upper_limit="${radians(90)}"
+      neck_pitch_upper_limit="${radians(55)}"
       neck_joints_effort_limit="${EFFORT_LIMIT}"
       neck_joints_velocity_limit="${VELOCITY_LIMIT}"
