Commit message: refactored robot and vehicle urdf files

File: sciurus17_description/robots/sciurus17.urdf.xacro (robot description, xacro)
@@ -1,5 +1,12 @@
 <?xml version="1.0"?>
 <robot name="sciurus17" xmlns:xacro="http://ros.org/wiki/xacro" >
+  <xacro:include filename="$(find sciurus17_description)/urdf/common_properties.xacro"/>
   <xacro:include filename="$(find sciurus17_description)/urdf/sciurus17/sciurus17_robot.urdf.xacro"/>
+  <!-- Used for fixing robot 'base_link'  to Gazebo 'world' -->
+  <link name="world"/>
+  <joint name="base_link_to_world_joint" type="fixed">
+    <parent link="world"/>
+    <child link="base_link"/>
+  </joint>
   <xacro:sciurus17_robot name="sciurus17_robot"/>
 </robot>

File: sciurus17_description/urdf/sciurus17/sciurus17_robot.urdf.xacro (robot description, xacro)
@@ -7,10 +7,4 @@
   <xacro:include filename="$(find sciurus17_description)/urdf/sciurus17/sciurus17_left_arm.xacro"/>
   <xacro:include filename="$(find sciurus17_description)/urdf/sciurus17/sciurus17_left_hand.xacro"/>
-  <material name="white">
-    <color rgba="0.9 0.9 0.9 1.0"/>
-  </material>
-  <material name="red">
-    <color rgba="0.8984375 0.0 0.0703125 1"/>
-  </material>
   <xacro:property name="EFFORT_LIMIT" value="4.0"/>
   <xacro:property name="VELOCITY_LIMIT" value="5.969211435"/>
@@ -58,10 +52,4 @@
       </xacro:if>
     </xacro:if>
-    <!-- Used for fixing robot 'base_link'  to Gazebo 'world' -->
-    <link name="world"/>
-    <joint name="base_link_to_world_joint" type="fixed">
-      <parent link="world"/>
-      <child link="base_link"/>
-    </joint>
     <xacro:sciurus17_body
       waist_yaw_upper_limit="${radians(-110)}"
