Commit message: added second laser scanner to urdf and srdf files

File: sciurus17_description/urdf/vehicle/sciurus_vehicle.gazebo.xacro (robot description, xacro)
@@ -197,5 +197,5 @@
     </plugin>
   </gazebo>
-  <gazebo reference="base_scan">
+  <gazebo reference="base_scan_front">
     <material>Gazebo/FlatBlack</material>
     <sensor type="ray" name="lds_lfcd_sensor">
@@ -225,9 +225,43 @@
       </ray>
       <plugin name="gazebo_ros_lds_lfcd_controller" filename="libgazebo_ros_laser.so">
-        <topicName>scan</topicName>
-        <frameName>base_scan</frameName>
+        <topicName>base_scan_front</topicName>
+        <frameName>base_scan_front</frameName>
         <update_rate>10</update_rate>
       </plugin>
     </sensor>
   </gazebo>
+  <gazebo reference="base_scan_back">
+    <material>Gazebo/FlatBlack</material>
+    <sensor type="ray" name="lds_lfcd_sensor">
+      <always_on>true</always_on>
+      <update_rate>10</update_rate>
+      <pose>0 0 0 0 0 0</pose>
+      <visualize>$(arg laser_visual)</visualize>
+      <ray>
+        <scan>
+          <horizontal>
+            <samples>485</samples>
+            <resolution>1.0</resolution>
+            <min_angle>-1.4848934412002563</min_angle>
+            <max_angle>1.4848934412002563</max_angle>
+          </horizontal>
+        </scan>
+        <range>
+          <min>0.06</min>
+          <max>6.0</max>
+          <resolution>0.01</resolution>
+        </range>
+        <noise>
+          <type>gaussian</type>
+          <mean>0.0</mean>
+          <stddev>0.01</stddev>
+        </noise>
+      </ray>
+      <plugin name="gazebo_ros_lds_lfcd_controller" filename="libgazebo_ros_laser.so">
+        <topicName>base_scan_back</topicName>
+        <frameName>base_scan_back</frameName>
+        <update_rate>10</update_rate>
+      </plugin>
+    </sensor>
+  </gazebo>
 </robot>

File: sciurus17_description/urdf/vehicle/sciurus_vehicle.urdf.xacro (robot description, xacro)
@@ -269,10 +269,10 @@
     </joint>
     <link name="imu_link"/>
-    <joint name="scan_joint" type="fixed">
-      <parent link="vehicle_base_link"/>
-      <child link="base_scan"/>
-      <origin xyz="0 0 0.1" rpy="0 0 0"/>
-    </joint>
-    <link name="base_scan">
+    <joint name="scan_joint_front" type="fixed">
+      <parent link="vehicle_base_link"/>
+      <child link="base_scan_front"/>
+      <origin xyz="-0.02 0 0.1" rpy="0 0 0"/>
+    </joint>
+    <link name="base_scan_front">
       <visual>
         <origin xyz="0 0 0" rpy="0 0 0"/>
@@ -296,4 +296,31 @@
       </inertial>
     </link>
+    <joint name="scan_joint_back" type="fixed">
+      <parent link="vehicle_base_link"/>
+      <child link="base_scan_back"/>
+      <origin xyz="-0.36 0 0.1" rpy="0 0 -3.14"/>
+    </joint>
+    <link name="base_scan_back">
+      <visual>
+        <origin xyz="0 0 0" rpy="0 0 0"/>
+        <geometry>
+          <mesh filename="package://sciurus17_description/meshes/vehicle/sensors/hokuyo.dae"/>
+        </geometry>
+        <material name="dark"/>
+      </visual>
+      <collision>
+        <origin xyz="0 0 0" rpy="0 0 0" />
+        <geometry>
+          <mesh filename="package://sciurus17_description/meshes/vehicle/sensors/hokuyo_convex.dae" />
+        </geometry>
+      </collision>
+      <inertial>
+        <mass value="0.114" />
+        <origin xyz="0 0 0" />
+        <inertia ixx="0.0" ixy="0.0" ixz="0.0"
+                 iyy="0.0" iyz="0.0"
+                 izz="0.0" />
+      </inertial>
+    </link>
     <joint name="sciurus17_joint" type="fixed">
       <parent link="base_footprint"/>
